File: pcb/keygen.kicad_pcb (KiCad board)
At the start: 2 copper layers, 362.9 x 125.8 mm, 236 parts, among them J101 PJ-320A, J201 PJ-320A, SW101 =, SW102 1, SW103 2, SW104 3, SW105 4, SW106 5, SW107 Tab, SW108 Q, SW109 W, SW110 E, SW111 R, SW112 T, SW113 Esc, SW114 A, SW115 S, SW116 D, SW117 F, SW118 G, SW119 Alt, SW120 Shift, SW121 Z, SW122 X, SW123 C, SW124 V, SW125 B, SW126 Ctrl, SW127 `, SW128 Caps, SW129 Left, SW130 Right, SW131 Super, SW132 Bksp, SW133 Del, SW190 MSK12C02 power, SW191 Reset, SW201 -, SW202 0, SW203 9, SW204 8, SW205 7, SW206 6, SW208 \, SW209 P, SW210 O, SW211 I, SW212 U, SW213 Y, SW214 ', SW215 ;, SW216 L, SW217 K, SW218 J, SW219 H, SW220 Alt, SW221 Shift, SW222 /, SW223 ., SW224 ,, SW225 M, SW226 N, SW227 Ctrl, SW228 ], SW229 [, SW230 Down, SW231 Up, SW232 Fn, SW233 Space, SW234 Enter, SW290 MSK12C02 power, SW291 Reset, U101 nRF52840 Pro Micro, U201 nRF52840 Pro Micro

Commit message: Straighten routed tracks into 0/45/90 degree runs
tools/smooth_route.py string-pulls every track chain (one net, layer
and width between pads, vias and junctions) into straight and 45-degree
segments, checking clearance with KiCad's own collision, then refills
the zones and stitches back any ground piece a moved track cut off.
On the board: 5551 -> 3567 segments, plus one GND via on the right.

route_pcb.stitch_fragments shared its union-find keys between the left
and right GND nets, so a split right-half pour counted as connected
through the left half and never got its via; clear them per net.

DRC with schematic parity: 0 errors, 0 unconnected (22 silkscreen
warnings, as before).
Routing:
- net /left/COL6: track 121.8 -> 119.2 mm
- net /left/LED_D1: track 42.6 -> 40.0 mm
- net /right/ENC_A: track 61.8 -> 59.9 mm
- net /left/VCC: track 798.4 -> 796.5 mm
- net /right/VCC: track 838.3 -> 836.6 mm
- net /left/LED_D17: track 30.5 -> 29.6 mm
- net /left/COL3: track 176.7 -> 175.9 mm
- net /right/COL3: track 179.6 -> 178.9 mm
- net /right/LED_D27: track 15.1 -> 14.4 mm
- net /left/LED_D19: track 139.7 -> 139.0 mm
- net /right/GND: track 94.4 -> 95.0 mm, vias 198 -> 199
- net /left/LED_D14: track 45.5 -> 44.8 mm
- net /left/UART_RX: track 5.61 -> 5.02 mm
- net /right/LED_D18: track 51.2 -> 50.6 mm
- net /left/LED_D20: track 32.9 -> 32.3 mm
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