File: pcb/keygen.kicad_pcb (KiCad board)
At the start: 2 copper layers, 362.9 x 125.8 mm, 224 parts, among them J101 PJ-320A, J201 PJ-320A, SW101 =, SW102 1, SW103 2, SW104 3, SW105 4, SW106 5, SW107 Tab, SW108 Q, SW109 W, SW110 E, SW111 R, SW112 T, SW113 Esc, SW114 A, SW115 S, SW116 D, SW117 F, SW118 G, SW119 Alt, SW120 Shift, SW121 Z, SW122 X, SW123 C, SW124 V, SW125 B, SW126 Ctrl, SW127 `, SW128 Caps, SW129 Left, SW130 Right, SW131 Super, SW132 Bksp, SW133 Del, SW190 MSK12C02 power, SW191 Reset, SW201 -, SW202 0, SW203 9, SW204 8, SW205 7, SW206 6, SW208 \, SW209 P, SW210 O, SW211 I, SW212 U, SW213 Y, SW214 ', SW215 ;, SW216 L, SW217 K, SW218 J, SW219 H, SW220 Alt, SW221 Shift, SW222 /, SW223 ., SW224 ,, SW225 M, SW226 N, SW227 Ctrl, SW228 ], SW229 [, SW230 Down, SW231 Up, SW232 Fn, SW233 Space, SW234 Enter, SW290 MSK12C02 power, SW291 Reset, U101 nRF52840 Pro Micro, U201 nRF52840 Pro Micro

Commit message: Restore the antenna keep-outs and print the battery + on the board
Re-poured with the fixed route_pcb.py (cleanup_pcb.py twice: the second
pass removes two GND vias left dangling under U101's antenna once the
fill there is gone), then sync_pcb.py added the "+" beside pad 1 of
BT101/BT201. D234's "K" moves to the other side of its pad, off the
board edge.

DRC with schematic parity: 0 errors, 0 unconnected, 0 parity, 22
silkscreen warnings. check_datasheets.py: 93 pass, 10 warn, 0 fail. Its
battery "+" check matched "SilkS" in the layer name, which KiCad 10
reports as "B.Silkscreen", so it now compares the layer itself.
Gerbers regenerated.
Routing:
- net /left/GND: vias 196 -> 194
Other:
- board text added: "+"
