File: pcb/left.kicad_sch (KiCad schematic)
At the start: 116 parts, among them Q101 AO3401A, Q102 AO3401A, Q103 AO3400A, SW101 =, SW102 1, SW103 2, SW104 3, SW105 4, SW106 5, SW107 Tab, SW108 Q, SW109 W, SW110 E, SW111 R, SW112 T, SW113 Esc, SW114 A, SW115 S, SW116 D, SW117 F, SW118 G, SW119 Alt, SW120 Shift, SW121 Z, SW122 X, SW123 C, SW124 V, SW125 B, SW126 Ctrl, SW127 `, SW128 Caps, SW129 Left, SW130 Right, SW131 Super, SW132 Bksp, SW133 Del, SW190 MSK12C02 power, SW191 Reset, U101 nRF52840 Pro Micro

Commit message: Add the switch plate, the gasket-mounted case, two OLEDs and a second knob
Switch plate: a 1.6 mm FR-4 board with black mask and no copper, made by
the PCB fab. tools/gen_plate.py writes it as its own KiCad board
(pcb/plate/) with Gerbers per half and fab/PLATE.md. It follows the PCB
outline with eight gasket tabs per half, 14 mm switch cut-outs, an
encoder cut-out and an OLED window per half, and the M2 holes.

Case: a 3D-printed PETG bottom shell and top frame per half, written by
tools/gen_case.py (build123d) to case/ as STL and STEP. The plate and
PCB, tied by M2 standoffs, float on Poron strips above and below each
tab; eight M2 screws per half close the case into heat-set inserts. It
has an open USB-C slot, a power switch slot with the wall thinned in
front, and a guided reset pinhole. A fit check against the PCB, plate,
controller, reset button, OLEDs and keycaps at full travel finds no
overlaps. The floor stays flat until tenting is chosen. Shared geometry
is in tools/case_geometry.py; tools/render_case.py renders the case and
the plate.

Knobs and OLEDs: the right encoder moves 7.6 mm inward and 4.1 mm up,
from 0.5 mm to 8.1 mm clear of the nearest keycap, and a mirrored
encoder joins the left half (push at row 0 / column 6, which renumbers
the left keys after it to SW108-SW134 / D108-D134). Each half gets a
0.96 in. SSD1306 OLED (J101/J201) over the controller's lower end, on
P0.17/P0.20, powered from the nice!nano's switched VCC. Both encoders
move to P0.10/P0.09, so both halves share one pin map with every edge
pin in use. The left reset button moves 6.5 mm so both halves mirror.
The new parts were added to the routed board and rerouted locally with
finish_route.py and smooth_route.py; the artwork was redrawn.

Firmware: both encoders, ZMK's status screen on both OLEDs (blanking
when idle), P0.13 held high by a gpio-hog for the OLED's power, and
ext-power on P0.08 only. The left knob scrolls (Super + scroll walks
Hyprland's workspaces) and clicks the mid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
Parts:
- removed SW107: Tab, keygen:SW_MX_HS_CPG151101S11_1.25u, symbol marbastlib-mx:MX_SW_HS_CPG151101S11
- added D134: 1N4148, Diode_THT:D_DO-35_SOD27_P7.62mm_Horizontal, symbol Device:D
- added ENC101: EC11, keygen:ROT_Alps_EC11E-Switch, symbol Device:RotaryEncoder_Switch
- added J101: OLED 0.96in I2C, Connector_PinHeader_2.54mm:PinHeader_1x04_P2.54mm_Vertical, symbol Connector_Generic:Conn_01x04
- added SW134: Del, keygen:SW_MX_HS_CPG151101S11_1.5u, symbol marbastlib-mx:MX_SW_HS_CPG151101S11
- SW108: value Q -> Tab; footprint keygen:SW_MX_HS_CPG151101S11_1u -> keygen:SW_MX_HS_CPG151101S11_1.25u
- SW109: value W -> Q
- SW110: value E -> W
- SW111: value R -> E
- SW112: value T -> R
- SW113: value Esc -> T; footprint keygen:SW_MX_HS_CPG151101S11_1.25u -> keygen:SW_MX_HS_CPG151101S11_1u
- SW114: value A -> Esc; footprint keygen:SW_MX_HS_CPG151101S11_1u -> keygen:SW_MX_HS_CPG151101S11_1.25u
- SW115: value S -> A
- SW116: value D -> S
- SW117: value F -> D
- SW118: value G -> F
- SW119: value Alt -> G
- SW120: value Shift -> Alt; footprint keygen:SW_MX_HS_CPG151101S11_1.25u -> keygen:SW_MX_HS_CPG151101S11_1u
- SW121: value Z -> Shift; footprint keygen:SW_MX_HS_CPG151101S11_1u -> keygen:SW_MX_HS_CPG151101S11_1.25u
- SW122: value X -> Z
- SW123: value C -> X
- SW124: value V -> C
- SW125: value B -> V
- SW126: value Ctrl -> B
- SW127: value ` -> Ctrl
- SW128: value Caps -> `
- SW129: value Left -> Caps
- SW130: value Right -> Left
- SW131: value Super -> Right; footprint keygen:SW_MX_HS_CPG151101S11_1.25u -> keygen:SW_MX_HS_CPG151101S11_1u
- SW132: value Bksp -> Super; footprint keygen:SW_MX_HS_CPG151101S11_1.5u -> keygen:SW_MX_HS_CPG151101S11_1.25u
- SW133: value Del -> Bksp
Connections:
- net COL0: now also SW108.1, SW114.1, SW121.1, SW128.1; no longer SW113.1, SW120.1, SW127.1
- net COL1: now also SW109.1, SW115.1, SW122.1, SW129.1; no longer SW108.1, SW114.1, SW121.1, SW128.1
- net COL2: now also SW110.1, SW116.1, SW123.1, SW130.1; no longer SW109.1, SW115.1, SW122.1, SW129.1
- net COL3: now also SW111.1, SW117.1, SW124.1, SW131.1; no longer SW110.1, SW116.1, SW123.1, SW130.1
- net COL4: now also SW112.1, SW118.1, SW125.1, SW132.1; no longer SW111.1, SW117.1, SW124.1, SW131.1
- net COL5: now also SW113.1, SW119.1, SW126.1, SW133.1; no longer SW112.1, SW118.1, SW125.1, SW132.1
- net COL6: now also SW120.1, SW127.1, ENC101.S1, SW134.1; no longer SW119.1, SW126.1, SW133.1
- net GND: now also ENC101.C, J101.1 (Pin_1)
- net K10: now also D108.2 (A), SW108.2; no longer D107.2 (A)
- net K11: now also D109.2 (A), SW109.2; no longer D108.2 (A), SW108.2
- net K12: now also D110.2 (A), SW110.2; no longer D109.2 (A), SW109.2
- net K13: now also D111.2 (A), SW111.2; no longer D110.2 (A), SW110.2
- net K14: now also D112.2 (A), SW112.2; no longer D111.2 (A), SW111.2
- net K15: now also D113.2 (A), SW113.2; no longer D112.2 (A), SW112.2
- net K20: now also D114.2 (A), SW114.2; no longer D113.2 (A), SW113.2
- net K21: now also D115.2 (A), SW115.2; no longer D114.2 (A), SW114.2
- net K22: now also D116.2 (A), SW116.2; no longer D115.2 (A), SW115.2
- net K23: now also D117.2 (A), SW117.2; no longer D116.2 (A), SW116.2
- net K24: now also D118.2 (A), SW118.2; no longer D117.2 (A), SW117.2
- net K25: now also D119.2 (A), SW119.2; no longer D118.2 (A), SW118.2
- net K26: now also D120.2 (A), SW120.2; no longer D119.2 (A), SW119.2
- net K30: now also D121.2 (A), SW121.2; no longer D120.2 (A), SW120.2
- net K31: now also D122.2 (A), SW122.2; no longer D121.2 (A), SW121.2
- net K32: now also D123.2 (A), SW123.2; no longer D122.2 (A), SW122.2
- net K33: now also D124.2 (A), SW124.2; no longer D123.2 (A), SW123.2
- net K34: now also D125.2 (A), SW125.2; no longer D124.2 (A), SW124.2
- net K35: now also D126.2 (A), SW126.2; no longer D125.2 (A), SW125.2
- net K36: now also D127.2 (A), SW127.2; no longer D126.2 (A), SW126.2
- net K40: now also D128.2 (A), SW128.2; no longer D127.2 (A), SW127.2
- net K41: now also D129.2 (A), SW129.2; no longer D128.2 (A), SW128.2
- net K42: now also D130.2 (A), SW130.2; no longer D129.2 (A), SW129.2
- net K43: now also D131.2 (A), SW131.2; no longer D130.2 (A), SW130.2
- net K44: now also D132.2 (A), SW132.2; no longer D131.2 (A), SW131.2
- net K45: now also D133.2 (A), SW133.2; no longer D132.2 (A), SW132.2
- net K46: now also D134.2 (A), SW134.2; no longer D133.2 (A), SW133.2
- net ROW0: now also D107.1 (K)
- net ROW1: now also D113.1 (K); no longer D107.1 (K)
- net ROW2: now also D120.1 (K); no longer D113.1 (K)
- net ROW3: now also D127.1 (K); no longer D120.1 (K)
- net ROW4: now also D134.1 (K); no longer D127.1 (K)
- net VCC: now reaches U101.16 (VCC)
- net VCC: now also J101.2 (Pin_2)
- net ENC_A: now reaches U101.23 (P0.10)
- net ENC_A: now also ENC101.A
- net ENC_B: now reaches U101.24 (P0.09)
- net ENC_B: now also ENC101.B
- net OLED_SDA: now reaches U101.5 (P0.17)
- net OLED_SDA: now also J101.4 (Pin_4)
- net OLED_SCL: now reaches U101.6 (P0.20)
- net OLED_SCL: now also J101.3 (Pin_3)
- new net K06: D107.2 (A), ENC101.S2
- no-connect marks 6 -> 1
Other:
- note added: "Encoder A/B on P0.10/P0.09 (NFC pins): set nfct-pins-as-gpios. P0.08: LED power switch. P0.17/P0.20: OLED SDA/SCL. VCC (pad 16, switched by P0.13): OLED power; firmware holds P0.13 high."
- note added: "Encoder S1/S2 (see ENC101)"
- note added: "OLED (0.96 in. 128x64 SSD1306, I2C address 0x3C) - check the module's pin order: GND VCC SCL SDA"
- note added: "ROTARY ENCODER (EC11) - push switch in the matrix at ROW0/COL6"
- note removed: "P0.08: LED power switch. VCC (pad 16) unused. Spare: P0.17 (full speed), P0.20, P0.09, P0.10"
- moved on the sheet: D107, D108, D109, D110, D111, D112, D113, D114, D115, D116, D117, D118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
