File: pcb/right.kicad_sch (KiCad schematic)
At the start: 113 parts, among them J201 PJ-320A, SW201 -, SW202 0, SW203 9, SW204 8, SW205 7, SW206 6, SW208 \, SW209 P, SW210 O, SW211 I, SW212 U, SW213 Y, SW214 ', SW215 ;, SW216 L, SW217 K, SW218 J, SW219 H, SW220 Alt, SW221 Shift, SW222 /, SW223 ., SW224 ,, SW225 M, SW226 N, SW227 Ctrl, SW228 ], SW229 [, SW230 Down, SW231 Up, SW232 Fn, SW233 Space, SW234 Enter, SW290 MSK12C02 power, SW291 Reset, U201 nRF52840 Pro Micro

Commit message: Drop the TRRS jack and switch the battery through a MOSFET
Settle power and connectivity before ordering. The halves talk over
Bluetooth only; USB-C on the left half is the wired mode. The TRRS jack
would only have replaced the Bluetooth split, needs its own ZMK build,
can't charge the other half (the nice!nano has no VBUS pin) and must not
be hot-plugged while a half is powered, which with a battery in each half
is always. P0.08 and P0.17 become spare.

The genuine nice!nano v2 charges at 500 mA with BOOST bridged, but the
MSK12C02 slide switch is rated 50 mA. It now only drives the gate of an
AO3401A P-MOSFET (source on the battery, drain on B+) with a 1 MOhm gate
resistor, so no battery current passes through its contacts. The lever and
case opening are unchanged.

Battery: a pouch up to 5 mm thick, 1000-1500 mAh, lying over the hotswap
sockets under the inner columns, inside the depth the socketed controller
already needs.

DRC with schematic parity: 0 errors, 0 unconnected, 0 parity issues.
Datasheet audit: 85 pass, 8 warn, 0 fail.
Parts:
- removed J201: PJ-320A, keygen:TRRS-PJ-320A, symbol keygen:TRRS_PJ-320A
- added Q201: AO3401A, Package_TO_SOT_SMD:SOT-23, symbol Transistor_FET:AO3401A
- added R201: 1M, Resistor_SMD:R_0805_2012Metric, symbol Device:R
Connections:
- net BAT_RAW: now also SW290.3 (C), Q201.2 (S), R201.2; no longer SW290.1 (A)
- net GND: now also SW290.1 (A)
- net VBAT: now also Q201.3 (D); no longer SW290.2 (B)
- net UART_RX: no longer names the net of U201.5 (P0.17)
- net UART_TX: no longer names the net of U201.2 (P0.08)
- new net BAT_GATE: Q201.1 (G), R201.1, SW290.2 (B)
Other:
- note added: "BATTERY SWITCH (P-MOSFET; the slide switch only drives the gate)"
- note added: "Encoder B on P0.09 (NFC pin): set nfct-pins-as-gpios. Spare: P0.08, P0.17 (full speed), P0.10"
- note added: "Switch 2-1: gate to GND, on. Switch 2-3: gate to source, off. R1 holds the gate off between positions. Leave the switch on while charging: off, USB charges the cell through the body diode (~0.35 W at 500 mA)."
- note removed: "TRRS (optional wired split; GND/TX/RX only, never battery power)"
- note removed: "UART: tip = P0.08, ring1 = P0.17 on BOTH halves. Left firmware: tx P0.08 / rx P0.17. Right firmware: tx P0.17 / rx P0.08 (crossed in software). Encoder B on P0.09 (NFC pin): set nfct-pins-as-gpios. Spare: P0.10"
Changed lines of the file:
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@@
     (effects (font (size 1.27 1.27)) (justify right bottom))
   )
-  (label "UART_TX"
-    (at 347.98 48.26 180)
-    (effects (font (size 1.27 1.27)) (justify right bottom))
-  )
+  (no_connect (at 347.98 48.26))
   (label "GND"
     (at 347.98 50.8 180)
@@
     (effects (font (size 1.27 1.27)) (justify right bottom))
   )
-  (label "UART_RX"
-    (at 347.98 55.88 180)
-    (effects (font (size 1.27 1.27)) (justify right bottom))
-  )
+  (no_connect (at 347.98 55.88))
   (label "ENC_A"
     (at 347.98 58.42 180)
@@
     (effects (font (size 1.27 1.27)) (justify left bottom))
   )
-  (text "UART: tip = P0.08, ring1 = P0.17 on BOTH halves.\nLeft firmware: tx P0.08 / rx P0.17.\nRight firmware: tx P0.17 / rx P0.08 (crossed in software).\nEncoder B on P0.09 (NFC pin): set nfct-pins-as-gpios.\nSpare: P0.10"
+  (text "Encoder B on P0.09 (NFC pin): set nfct-pins-as-gpios.\nSpare: P0.08, P0.17 (full speed), P0.10"
     (exclude_from_sim no)
     (at 386.08 45.72 0)
@@
     )
   )
+  (label "GND"
+    (at 365.76 129.54 0)
+    (effects (font (size 1.27 1.27)) (justify left bottom))
+  )
+  (label "BAT_GATE"
+    (at 355.6 132.08 180)
+    (effects (font (size 1.27 1.27)) (justify right bottom))
+  )
   (label "BAT_RAW"
-    (at 365.76 129.54 0)
-    (effects (font (size 1.27 1.27)) (justify left bottom))
-  )
-  (label "VBAT"
-    (at 355.6 132.08 180)
-    (effects (font (size 1.27 1.27)) (justify right bottom))
-  )
-  (no_connect (at 365.76 134.62))
+    (at 365.76 134.62 0)
+    (effects (font (size 1.27 1.27)) (justify left bottom))
+  )
   (symbol
     (lib_id "Switch:SW_Push")
@@
     (effects (font (size 1.27 1.27)) (justify left top))
   )
-  (text "TRRS (optional wired split; GND/TX/RX only, never battery power)"
+  (text "BATTERY SWITCH (P-MOSFET; the slide switch only drives the gate)"
     (exclude_from_sim no)
     (at 335.28 170.18 0)
@@
   )
   (symbol
-    (lib_id "keygen:TRRS_PJ-320A")
+    (lib_id "Transistor_FET:AO3401A")
     (at 360.68 185.42 0)
     (unit 1)
@@
     (on_board yes)
     (dnp no)
-    (property "Reference" "J201" (at 360.68 179.07 0) (effects (font (size 1.27 1.27))))
-    (property "Value" "PJ-320A" (at 360.68 191.77 0) (effects (font (size 1.27 1.27))))
-    (property "Footprint" "keygen:TRRS-PJ-320A"
+    (property "Reference" "Q201" (at 360.68 179.07 0) (effects (font (size 1.27 1.27))))
+    (property "Value" "AO3401A" (at 360.68 191.77 0) (effects (font (size 1.27 1.27))))
+    (property "Footprint" "Package_TO_SOT_SMD:SOT-23"
       (at 360.68 185.42 0)
       (effects (font (size 1.27 1.27)) (hide yes))
     )
     (property "Datasheet" "" (at 360.68 185.42 0) (effects (font (size 1.27 1.27)) (hide yes)))
+    (pin "1")
     (pin "2")
     (pin "3")
-    (pin "4")
-    (pin "1")
-    (instances
-      (project "keygen"
-        (path "/6967da33-a0e5-5fa7-9742-40725aff3c90/0c428d53-712b-56dc-b044-5fe085247794"
-          (reference "J201")
-          (unit 1)
-        )
-      )
-    )
-  )
-  (label "UART_TX"
-    (at 365.76 182.88 0)
-    (effects (font (size 1.27 1.27)) (justify left bottom))
-  )
-  (label "UART_RX"
-    (at 365.76 185.42 0)
-    (effects (font (size 1.27 1.27)) (justify left bottom))
-  )
-  (no_connect (at 365.76 187.96))
-  (label "GND"
-    (at 365.76 190.5 0)
-    (effects (font (size 1.27 1.27)) (justify left bottom))
+    (instances
+      (project "keygen"
+        (path "/6967da33-a0e5-5fa7-9742-40725aff3c90/0c428d53-712b-56dc-b044-5fe085247794"
+          (reference "Q201")
+          (unit 1)
+        )
+      )
+    )
+  )
+  (label "BAT_GATE"
+    (at 355.6 185.42 180)
+    (effects (font (size 1.27 1.27)) (justify right bottom))
+  )
+  (label "BAT_RAW"
+    (at 363.22 190.5 270)
+    (effects (font (size 1.27 1.27)) (justify right bottom))
+  )
+  (label "VBAT"
+    (at 363.22 180.34 90)
+    (effects (font (size 1.27 1.27)) (justify left bottom))
+  )
+  (symbol
+    (lib_id "Device:R")
+    (at 375.92 185.42 0)
+    (unit 1)
+    (exclude_from_sim no)
+    (in_bom yes)
+    (on_board yes)
+    (dnp no)
+    (property "Reference" "R201" (at 375.92 179.07 0) (effects (font (size 1.27 1.27))))
+    (property "Value" "1M" (at 375.92 191.77 0) (effects (font (size 1.27 1.27))))
+    (property "Footprint" "Resistor_SMD:R_0805_2012Metric"
+      (at 375.92 185.42 0)
+      (effects (font (size 1.27 1.27)) (hide yes))
+    )
+    (property "Datasheet" "" (at 375.92 185.42 0) (effects (font (size 1.27 1.27)) (hide yes)))
+    (pin "1")
+    (pin "2")
+    (instances
+      (project "keygen"
+        (path "/6967da33-a0e5-5fa7-9742-40725aff3c90/0c428d53-712b-56dc-b044-5fe085247794"
+          (reference "R201")
+          (unit 1)
+        )
+      )
+    )
+  )
+  (label "BAT_GATE"
+    (at 375.92 181.61 90)
+    (effects (font (size 1.27 1.27)) (justify left bottom))
+  )
+  (label "BAT_RAW"
+    (at 375.92 189.23 270)
+    (effects (font (size 1.27 1.27)) (justify right bottom))
+  )
+  (text "Switch 2-1: gate to GND, on. Switch 2-3: gate to source, off.\nR1 holds the gate off between positions. Leave the switch on while charging:\noff, USB charges the cell through the body diode (~0.35 W at 500 mA)."
+    (exclude_from_sim no)
+    (at 335.28 198.12 0)
+    (effects (font (size 1.27 1.27)) (justify left top))
   )
   (text "ROTARY ENCODER (EC11) - push switch in the matrix at ROW0/COL6"

Commit message: Power the LEDs from the battery through a MOSFET switch
The SK6812MINI-E is rated for VDD 3.7-5.5 V, and the nice!nano's 3.3 V
VCC has no published current limit for 33 LEDs. The LED rail (LED_VDD)
now runs from B+ through an AO3401A P-MOSFET (Q2). An AO3400A N-MOSFET
(Q3) on P0.08 pulls Q2's gate low to turn the LEDs on; 100 kOhm
resistors hold Q2 off (R2, gate to source) and Q3 off while the
controller boots or sleeps (R3). The 10 uF + 100 nF capacitors move to
Q2's output. VCC (pad 16) is unused. The cell is inside the LEDs'
rating until it runs low, and they light only on USB power.

All resistors and capacitors are now 1206 hand-solder footprints. The
new parts sit on the back between each battery connector and the board
edge, clear of the mounting holes, the antenna end and the top-edge
slot. They were added to the routed board, which was rerouted locally
with finish_route.py and smooth_route.py; the artwork was redrawn.

Firmware: ZMK's ext-power now drives P0.08 (and still P0.13, which only
switches the unused VCC). All three UF2 builds pass.

DRC with schematic parity: 0 errors, 0 unconnected, 0 parity; 14
silkscreen warnings. check_datasheets.py: 100 pass, 8 warn, 0 fail.
Parts:
- added Q202: AO3401A, Package_TO_SOT_SMD:SOT-23, symbol Transistor_FET:AO3401A
- added Q203: AO3400A, Package_TO_SOT_SMD:SOT-23, symbol Transistor_FET:AO3400A
- added R202, R203: 100k, Resistor_SMD:R_1206_3216Metric_Pad1.30x1.75mm_HandSolder, symbol Device:R
- BT201: value LiPo 3.7V ~1000mAh -> LiPo 3.7V 3000mAh
- C201, C202: footprint Capacitor_SMD:C_0805_2012Metric -> Capacitor_SMD:C_1206_3216Metric_Pad1.33x1.80mm_HandSolder
- R201: footprint Resistor_SMD:R_0805_2012Metric -> Resistor_SMD:R_1206_3216Metric_Pad1.30x1.75mm_HandSolder
Connections:
- net GND: now also Q203.2 (S), R203.2
- net VBAT: now also Q202.2 (S), R202.2
- net LED_EN: now reaches U201.2 (P0.08)
- net LED_EN: now also Q203.1 (G), R203.1
- net VCC renamed LED_VDD
- net LED_VDD: now also Q202.3 (D); no longer U201.16 (VCC)
- new net LED_GATE: Q202.1 (G), Q203.3 (D), R202.1
Other:
- note added: "C1/C2 sit at the LED power switch's output."
- note added: "Encoder B on P0.09 (NFC pin): set nfct-pins-as-gpios. P0.08: LED power switch. VCC (pad 16) unused. Spare: P0.17 (full speed), P0.10"
- note added: "LED POWER SWITCH (P0.08 high = LEDs on)"
- note added: "PER-KEY LEDs (33) - powered from the battery through the LED power switch (Q2, LED_VDD)"
- note removed: "C1/C2 sit next to the first LED of the chain."
- note removed: "Encoder B on P0.09 (NFC pin): set nfct-pins-as-gpios. Spare: P0.08, P0.17 (full speed), P0.10"
- note removed: "PER-KEY LEDs (33, no underglow) - powered from the controller's switched VCC (P0.13); cap brightness in firmware"
