File: pcb/plate/keygen-plate.kicad_pcb (KiCad board)
At the start: 2 copper layers, 372.9 x 130.9 mm, 10 parts

Commit message: Lower both knobs 4 mm and size them for a 17 x 13 mm knob
Both encoder shafts move 4 mm toward the thumbs (y 125 to 129), so the
knob no longer sits against the OLED and is closer to the thumb. With a
17 mm knob its edge is 4.5 mm below the OLED module, 5.7 mm from the
thumb cluster's top key and 9.1 mm from the G/H column. The encoder
diodes stay where they were, beside the switch pins.

The encoders' tracks were ripped and rerouted with finish_route.py and
smooth_route.py; the artwork was redrawn. Each EC11's common pin C,
2.5 mm between A and B, now connects to the ground pour solid: there is
no room for thermal spokes beside it.

The knob model is now 17 x 13 mm (an "amplifier" knob, D half shaft),
and the plate, case, plate print, ZMK physical layout, keymap pictures,
renders and docs follow. All three UF2 builds pass.

DRC with schematic parity: 0 errors, 0 unconnected, 0 parity; 16
silkscreen warnings. check_schematic.py clean. check_datasheets.py: 107
pass, 11 warn, 0 fail. Case fit check: no overlaps.
Other:
- outline, holes or cut-outs redrawn
Changed lines of the file:
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@@
   (footprint "MountingHole:MountingHole_2.2mm_M2"
     (layer "F.Cu")
-    (at 241.5499 88.5757)
+    (at 34.794 161.0757)
     (descr "Mounting Hole 2.2mm, M2, no annular, generated by kicad-footprint-generator mountinghole.py"
     )
     (tags "mountinghole M2")
-    (property "Reference" "H202"
+    (property "Reference" "H102"
       (at 0 -3.15 0)
       (layer "F.SilkS")
@@
   (footprint "MountingHole:MountingHole_2.2mm_M2"
     (layer "F.Cu")
-    (at 114.294 135.5757)
+    (at 182.294 89.0757)
     (descr "Mounting Hole 2.2mm, M2, no annular, generated by kicad-footprint-generator mountinghole.py"
     )
     (tags "mountinghole M2")
-    (property "Reference" "H101"
+    (property "Reference" "H103"
       (at 0 -3.15 0)
       (layer "F.SilkS")
@@
   (footprint "MountingHole:MountingHole_2.2mm_M2"
     (layer "F.Cu")
-    (at 315.0499 133.0757)
+    (at 53.794 84.0757)
     (descr "Mounting Hole 2.2mm, M2, no annular, generated by kicad-footprint-generator mountinghole.py"
     )
     (tags "mountinghole M2")
-    (property "Reference" "H201"
+    (property "Reference" "H105"
       (at 0 -3.15 0)
       (layer "F.SilkS")
@@
   (footprint "MountingHole:MountingHole_2.2mm_M2"
     (layer "F.Cu")
-    (at 258.049899 194.0757)
+    (at 114.294 135.5757)
     (descr "Mounting Hole 2.2mm, M2, no annular, generated by kicad-footprint-generator mountinghole.py"
     )
     (tags "mountinghole M2")
-    (property "Reference" "H203"
+    (property "Reference" "H101"
       (at 0 -3.15 0)
       (layer "F.SilkS")
@@
   (footprint "MountingHole:MountingHole_2.2mm_M2"
     (layer "F.Cu")
-    (at 182.294 89.0757)
+    (at 388.5499 161.0757)
     (descr "Mounting Hole 2.2mm, M2, no annular, generated by kicad-footprint-generator mountinghole.py"
     )
     (tags "mountinghole M2")
-    (property "Reference" "H103"
+    (property "Reference" "H204"
       (at 0 -3.15 0)
       (layer "F.SilkS")
@@
   (footprint "MountingHole:MountingHole_2.2mm_M2"
     (layer "F.Cu")
-    (at 34.794 161.0757)
+    (at 241.5499 88.5757)
     (descr "Mounting Hole 2.2mm, M2, no annular, generated by kicad-footprint-generator mountinghole.py"
     )
     (tags "mountinghole M2")
-    (property "Reference" "H102"
+    (property "Reference" "H202"
       (at 0 -3.15 0)
       (layer "F.SilkS")
@@
   (footprint "MountingHole:MountingHole_2.2mm_M2"
     (layer "F.Cu")
-    (at 166.294 196.5757)
+    (at 315.0499 133.0757)
     (descr "Mounting Hole 2.2mm, M2, no annular, generated by kicad-footprint-generator mountinghole.py"
     )
     (tags "mountinghole M2")
-    (property "Reference" "H104"
+    (property "Reference" "H201"
       (at 0 -3.15 0)
       (layer "F.SilkS")
@@
   (footprint "MountingHole:MountingHole_2.2mm_M2"
     (layer "F.Cu")
-    (at 53.794 84.0757)
+    (at 258.049899 194.0757)
     (descr "Mounting Hole 2.2mm, M2, no annular, generated by kicad-footprint-generator mountinghole.py"
     )
     (tags "mountinghole M2")
-    (property "Reference" "H105"
+    (property "Reference" "H203"
       (at 0 -3.15 0)
       (layer "F.SilkS")
@@
   (footprint "MountingHole:MountingHole_2.2mm_M2"
     (layer "F.Cu")
-    (at 388.5499 161.0757)
+    (at 166.294 196.5757)
     (descr "Mounting Hole 2.2mm, M2, no annular, generated by kicad-footprint-generator mountinghole.py"
     )
     (tags "mountinghole M2")
-    (property "Reference" "H204"
+    (property "Reference" "H104"
       (at 0 -3.15 0)
       (layer "F.SilkS")
@@
   )
   (gr_arc
-    (start 160.475 119)
-    (mid 160.621446 118.646446)
-    (end 160.975 118.5)
-    (stroke (width 0.05) (type default))
-    (layer "Edge.Cuts")
-  )
-  (gr_line
-    (start 160.475 131)
-    (end 160.475 119)
+    (start 160.475 123)
+    (mid 160.621446 122.646446)
+    (end 160.975 122.5)
+    (stroke (width 0.05) (type default))
+    (layer "Edge.Cuts")
+  )
+  (gr_line
+    (start 160.475 135)
+    (end 160.475 123)
     (stroke (width 0.05) (type default))
     (layer "Edge.Cuts")
@@
   )
   (gr_line
-    (start 160.975 118.5)
-    (end 172.975 118.5)
-    (stroke (width 0.05) (type default))
-    (layer "Edge.Cuts")
-  )
-  (gr_arc
-    (start 160.975 131.5)
-    (mid 160.621446 131.353553)
-    (end 160.475 131)
+    (start 160.975 122.5)
+    (end 172.975 122.5)
+    (stroke (width 0.05) (type default))
+    (layer "Edge.Cuts")
+  )
+  (gr_arc
+    (start 160.975 135.5)
+    (mid 160.621446 135.353553)
+    (end 160.475 135)
     (stroke (width 0.05) (type default))
     (layer "Edge.Cuts")
@@
   )
   (gr_arc
-    (start 172.975 118.5)
-    (mid 173.328553 118.646446)
-    (end 173.475 119)
-    (stroke (width 0.05) (type default))
-    (layer "Edge.Cuts")
-  )
-  (gr_line
-    (start 172.975 131.5)
-    (end 160.975 131.5)
-    (stroke (width 0.05) (type default))
-    (layer "Edge.Cuts")
-  )
-  (gr_line
-    (start 173.475 119)
-    (end 173.475 131)
-    (stroke (width 0.05) (type default))
-    (layer "Edge.Cuts")
-  )
-  (gr_arc
-    (start 173.475 131)
-    (mid 173.328553 131.353553)
-    (end 172.975 131.5)
+    (start 172.975 122.5)
+    (mid 173.328553 122.646446)
+    (end 173.475 123)
+    (stroke (width 0.05) (type default))
+    (layer "Edge.Cuts")
+  )
+  (gr_line
+    (start 172.975 135.5)
+    (end 160.975 135.5)
+    (stroke (width 0.05) (type default))
+    (layer "Edge.Cuts")
+  )
+  (gr_line
+    (start 173.475 123)
+    (end 173.475 135)
+    (stroke (width 0.05) (type default))
+    (layer "Edge.Cuts")
+  )
+  (gr_arc
+    (start 173.475 135)
+    (mid 173.328553 135.353553)
+    (end 172.975 135.5)
     (stroke (width 0.05) (type default))
     (layer "Edge.Cuts")
@@
   )
   (gr_arc
-    (start 250 119)
-    (mid 250.146446 118.646446)
-    (end 250.5 118.5)
-    (stroke (width 0.05) (type default))
-    (layer "Edge.Cuts")
-  )
-  (gr_line
-    (start 250 131)
-    (end 250 119)
-    (stroke (width 0.05) (type default))
-    (layer "Edge.Cuts")
-  )
-  (gr_line
-    (start 250.5 118.5)
-    (end 262.5 118.5)
-    (stroke (width 0.05) (type default))
-    (layer "Edge.Cuts")
-  )
-  (gr_arc
-    (start 250.5 131.5)
-    (mid 250.146446 131.353553)
-    (end 250 131)
+    (start 250 123)
+    (mid 250.146446 122.646446)
+    (end 250.5 122.5)
+    (stroke (width 0.05) (type default))
+    (layer "Edge.Cuts")
+  )
+  (gr_line
+    (start 250 135)
+    (end 250 123)
+    (stroke (width 0.05) (type default))
+    (layer "Edge.Cuts")
+  )
+  (gr_line
+    (start 250.5 122.5)
+    (end 262.5 122.5)
+    (stroke (width 0.05) (type default))
+    (layer "Edge.Cuts")
+  )
+  (gr_arc
+    (start 250.5 135.5)
+    (mid 250.146446 135.353553)
+    (end 250 135)
     (stroke (width 0.05) (type default))
     (layer "Edge.Cuts")
@@
   )
   (gr_arc
-    (start 262.5 118.5)
-    (mid 262.853553 118.646446)
-    (end 263 119)
-    (stroke (width 0.05) (type default))
-    (layer "Edge.Cuts")
-  )
-  (gr_line
-    (start 262.5 131.5)
-    (end 250.5 131.5)
+    (start 262.5 122.5)
+    (mid 262.853553 122.646446)
+    (end 263 123)
+    (stroke (width 0.05) (type default))
+    (layer "Edge.Cuts")
+  )
+  (gr_line
+    (start 262.5 135.5)
+    (end 250.5 135.5)
     (stroke (width 0.05) (type default))
     (layer "Edge.Cuts")
@@
   )
   (gr_line
-    (start 263 119)
-    (end 263 131)
-    (stroke (width 0.05) (type default))
-    (layer "Edge.Cuts")
-  )
-  (gr_arc
-    (start 263 131)
-    (mid 262.853553 131.353553)
-    (end 262.5 131.5)
-    (stroke (width 0.05) (type default))
-    (layer "Edge.Cuts")
+    (start 263 123)
+    (end 263 135)
+    (stroke (width 0.05) (type default))
+    (layer "Edge.Cuts")
+  )
+  (gr_arc
+    (start 263 135)
+    (mid 262.853553 135.353553)
+    (end 262.5 135.5)
+    (stroke (width 0.05) (type default))
+    (layer "Edge.Cuts")
