File: pcb/plate/keygen-plate.kicad_pcb (KiCad board)
At the start: 2 copper layers, 372.9 x 130.9 mm, 10 parts

Commit message: feat(layout): refine thumb cluster and OLED placement
Use 1.25u lower thumb keys, keep the upper pair at 1u, move the encoders and OLEDs, and align the board outline with the thumb row. Regenerate the routed PCB, case, plate, print sheets, fabrication files, BOM, and documentation.
Parts:
- moved H202 38.4 mm to (240.5, 127.0)
- moved H103 37.9 mm to (183.0, 127.0)
- moved H203 9.80 mm to (267.4, 191.0)
- moved H104 0.32 mm to (166.4, 196.9)
Other:
- board size 372.9 x 130.9 mm -> 372.9 x 130.5 mm
